File: Barometer-Pi-Module.kicad_pcb (KiCad board)
At the start: 2 copper layers, 27.9 x 15.2 mm, 13 parts, among them J1 Conn_01x05, J2 Conn_02x03_Odd_Even, J4 Conn_01x05, U1 MS560702BA03-50

Commit message: Tidy silk
Other:
- board text added: "I²C Barometer/ Altimeter"
- board text added: "Rev A 20181110"
- board text removed: "I²C Barometer Rev A 20181110"
